Commit message: 新增了奖励函数项

File: y2_isaacgym/resources/y2/urdf/robot.urdf (robot description, URDF)
Before this commit: robot Y2_dual_urdf_v0, 17 links, 16 joints
Links:
- added link imu_link, mass 0.001; collision box size=0.000518 0.000518 0.000518; visual box size=0.001 0.001 0.001
Joints:
- added joint imu_joint: type fixed, parent base_link, child imu_link, origin xyz=0 0 0 rpy=0 0 0
