Commit message: 和上面的一致

File: y2_isaacgym/resources/y2/urdf/robot18.urdf (robot description, URDF)
Before this commit: robot y2_description, 18 links, 17 joints
Joints:
- joint back_left_knee_joint: limit lower=-1.9199 upper=0 effort=80 velocity=15 -> lower=-1.9199 upper=0 effort=24 velocity=6; origin xyz=0.14 0 0 rpy=0 0 2.5197 -> xyz=0.18 0 0 rpy=0 0 2.5197
- joint back_left_thigh_joint: limit lower=-2.3562 upper=2.3562 effort=80 velocity=15 -> lower=-2.3562 upper=2.3562 effort=24 velocity=6
- joint back_left_wheel_joint: origin xyz=0.14 0 0 rpy=0 0 2.9781 -> xyz=0.18 0 0 rpy=0 0 2.9781
- joint back_right_knee_joint: limit lower=-1.9199 upper=0 effort=80 velocity=15 -> lower=-1.9199 upper=0 effort=24 velocity=6; origin xyz=0.14 0 0 rpy=0 0 2.5197 -> xyz=0.18 0 0 rpy=0 0 2.5197
- joint back_right_thigh_joint: limit lower=-2.3562 upper=2.3562 effort=80 velocity=15 -> lower=-2.3562 upper=2.3562 effort=24 velocity=6
- joint back_right_wheel_joint: origin xyz=0.14 0 0 rpy=0 0 2.9781 -> xyz=0.18 0 0 rpy=0 0 2.9781
- joint front_left_knee_joint: limit lower=0 upper=1.9199 effort=80 velocity=15 -> lower=0 upper=1.9199 effort=24 velocity=6; origin xyz=0.14 0 0 rpy=0 0 -2.5197 -> xyz=0.18 0 0 rpy=0 0 -2.5197
- joint front_left_thigh_joint: limit lower=-2.3562 upper=2.3562 effort=80 velocity=15 -> lower=-2.3562 upper=2.3562 effort=24 velocity=6
- joint front_left_wheel_joint: origin xyz=0.14 0 0 rpy=0 0 0.16348 -> xyz=0.18 0 0 rpy=0 0 0.16348
- joint front_right_knee_joint: limit lower=0 upper=1.9199 effort=80 velocity=15 -> lower=0 upper=1.9199 effort=24 velocity=6; origin xyz=0.14 0 0 rpy=0 0 -2.5197 -> xyz=0.18 0 0 rpy=0 0 -2.5197
- joint front_right_thigh_joint: limit lower=-2.3562 upper=2.3562 effort=80 velocity=15 -> lower=-2.3562 upper=2.3562 effort=24 velocity=6
- joint front_right_wheel_joint: origin xyz=0.14 0 0 rpy=0 0 0.16348 -> xyz=0.18 0 0 rpy=0 0 0.16348
